Commit message: J3 fix and std coordinates

File: yk400xe_description/urdf/joints.xacro (robot description, xacro)
@@ -23,7 +23,7 @@
         <parent link="L3"/>
         <child  link="L4_dummy"/>
-        <origin xyz="0 0.175 -0.068402" rpy="0 0 0"/>   <!-- check z TODO -->
+        <origin xyz="0 0.175 -0.063402" rpy="0 0 0"/>
         <axis xyz="0 0 1"/>
-        <limit effort="1000.0" lower="-0.150" upper="0" velocity="0.5"/>    <!-- 0 - 150 mm in -z  -->
+        <limit effort="1000.0" lower="-0.150" upper="0.00875" velocity="0.5"/>    <!-- 0 - 150 mm in -z  -->
     </joint>
     <joint name="J4" type="revolute">

File: yk400xe_description/urdf/yk400xe.urdf.xacro (robot description, xacro)
@@ -9,3 +9,9 @@
     <xacro:include filename="$(find yk400xe_description)/urdf/links.xacro" />
     <xacro:include filename="$(find yk400xe_description)/urdf/joints.xacro" />
+    <link name="std_coords_link"/>
+    <joint name="std_coords_joint">
+        <parent link="L1" type=fixed>
+        <child link="std_coords_link">
+        <origin xyz="0.0 0.0 0.0" rpy="0 0 0"/>  <!-- TODO z-->
+    <joint/>
 </robot>

Commit message: Fix and clean up
- Fixed error in trajectory commands creation
- Fixed URDF

File: yk400xe_description/urdf/joints.xacro (robot description, xacro)
@@ -24,6 +24,6 @@
         <child  link="L4_dummy"/>
         <origin xyz="0 0.175 -0.063402" rpy="0 0 0"/>
-        <axis xyz="0 0 1"/>
-        <limit effort="1000.0" lower="-0.150" upper="0.00875" velocity="0.5"/>    <!-- 0 - 150 mm in -z  -->
+        <axis xyz="0 0 -1"/>
+        <limit effort="1000.0" lower="-0.00875" upper="0.150" velocity="0.5"/>    <!-- -0.00875 - 150 mm in -z  -->
     </joint>
     <joint name="J4" type="revolute">
